File: picopad-v01/picopad-v01.kicad_pcb (KiCad board)
At the start: 2 copper layers, 0 parts

Commit message: Place the footprints on the PCB
Parts:
- added C1: 22pF, Capacitor_SMD:C_0805_2012Metric, B.Cu at (167.6, 137.3)
- added C10: 0.1uF, Capacitor_SMD:C_0603_1608Metric, B.Cu at (126.7, 64.2)
- added C11: 0.1uF, Capacitor_SMD:C_0603_1608Metric, B.Cu at (107.6, 64.2)
- added C12: 0.1uF, Capacitor_SMD:C_0603_1608Metric, B.Cu at (107.7, 83.2)
- added C13: 0.1uF, Capacitor_SMD:C_0603_1608Metric, B.Cu at (126.6, 83.2)
- added C14: 0.1uF, Capacitor_SMD:C_0603_1608Metric, B.Cu at (145.7, 83.2)
- added C15: 0.1uF, Capacitor_SMD:C_0603_1608Metric, B.Cu at (164.8, 92.7)
- added C16: 0.1uF, Capacitor_SMD:C_0603_1608Metric, B.Cu at (145.7, 102.3)
- added C17: 0.1uF, Capacitor_SMD:C_0603_1608Metric, B.Cu at (126.6, 102.3)
- added C18: 0.1uF, Capacitor_SMD:C_0603_1608Metric, B.Cu at (107.6, 102.3)
- added C19: 0.1uF, Capacitor_SMD:C_0603_1608Metric, B.Cu at (107.6, 121.3)
- added C2: 10uF, Capacitor_SMD:C_0805_2012Metric, B.Cu at (162.6, 92.8)
- added C20: 0.1uF, Capacitor_SMD:C_0603_1608Metric, B.Cu at (126.6, 121.3)
- added C21: 0.1uF, Capacitor_SMD:C_0603_1608Metric, B.Cu at (145.7, 121.3)
- added C22: 0.1uF, Capacitor_SMD:C_0603_1608Metric, B.Cu at (164.7, 130.9)
- added C23: 0.1uF, Capacitor_SMD:C_0603_1608Metric, B.Cu at (145.7, 140.4)
- added C24: 0.1uF, Capacitor_SMD:C_0603_1608Metric, B.Cu at (117.2, 140.3)
- added C3: 0.1uF, Capacitor_SMD:C_0805_2012Metric, B.Cu at (178.8, 96.0)
- added C4: 0.1uF, Capacitor_SMD:C_0805_2012Metric, B.Cu at (157.8, 106.2)
- added C5: 0.1uF, Capacitor_SMD:C_0805_2012Metric, B.Cu at (167.7, 119.0)
- added C6: 22pF, Capacitor_SMD:C_0805_2012Metric, B.Cu at (174.0, 137.3)
- added C7: 1uF, Capacitor_SMD:C_0805_2012Metric, B.Cu at (179.8, 106.1)
- added C8: 0.1uF, Capacitor_SMD:C_0603_1608Metric, B.Cu at (164.8, 64.2)
- added C9: 0.1uF, Capacitor_SMD:C_0603_1608Metric, B.Cu at (145.8, 64.2)
- added D1: SOD123, Diode_SMD:D_SOD-123, B.Cu at (176.9, 63.4)
- added D10: SOD123, Diode_SMD:D_SOD-123, B.Cu at (138.8, 101.5)
- added D11: SOD123, Diode_SMD:D_SOD-123, B.Cu at (119.7, 101.5)
- added D12: SOD123, Diode_SMD:D_SOD-123, B.Cu at (119.7, 120.4)
- added D13: SOD123, Diode_SMD:D_SOD-123, B.Cu at (138.8, 120.4)
- added D14: SOD123, Diode_SMD:D_SOD-123, B.Cu at (157.8, 120.4)
- added D15: SOD123, Diode_SMD:D_SOD-123, B.Cu at (176.9, 130.0)
- added D16: SOD123, Diode_SMD:D_SOD-123, B.Cu at (157.8, 139.5)
- added D17: SOD123, Diode_SMD:D_SOD-123, B.Cu at (129.2, 139.5)
- added D2: SOD123, Diode_SMD:D_SOD-123, B.Cu at (157.8, 63.4)
- added D3: SOD123, Diode_SMD:D_SOD-123, B.Cu at (138.8, 63.3)
- added D4: SOD123, Diode_SMD:D_SOD-123, B.Cu at (119.7, 63.3)
- added D5: SOD123, Diode_SMD:D_SOD-123, B.Cu at (119.7, 82.3)
- added D6: SOD123, Diode_SMD:D_SOD-123, B.Cu at (138.8, 82.3)
- added D7: SOD123, Diode_SMD:D_SOD-123, B.Cu at (157.8, 82.4)
- added D8: SOD123, Diode_SMD:D_SOD-123, B.Cu at (176.9, 91.9)
- added D9: SOD123, Diode_SMD:D_SOD-123, B.Cu at (157.8, 101.4)
- added F1: 500mA, Fuse:Fuse_1206_3216Metric, B.Cu at (121.6, 58.0)
- added MX1: NUMPAD_MINUS, picopad:MXOnly-1U-Hotswap, F.Cu at (171.0, 58.7)
- added MX10: NUMPAD_5, picopad:MXOnly-1U-Hotswap, F.Cu at (132.9, 96.8)
- added MX11: NUMPAD_4, picopad:MXOnly-1U-Hotswap, F.Cu at (113.9, 96.8)
- added MX12: NUMPAD_1, picopad:MXOnly-1U-Hotswap, F.Cu at (113.9, 115.8)
- added MX13: NUMPAD_2, picopad:MXOnly-1U-Hotswap, F.Cu at (132.9, 115.8)
- added MX14: NUMPAD_3, picopad:MXOnly-1U-Hotswap, F.Cu at (152.0, 115.8)
- added MX15: NUMPAD_ENTER, picopad:MXOnly-2U-Hotswap-Vertical, F.Cu at (171.0, 125.4)
- added MX16: NUMPAD_DOT, picopad:MXOnly-1U-Hotswap, F.Cu at (152.0, 134.9)
- added MX17: NUMPAD_0, picopad:MXOnly-2U-Hotswap, F.Cu at (123.4, 134.8)
- added MX2: NUMPAD_ASTERISK, picopad:MXOnly-1U-Hotswap, F.Cu at (152.0, 58.7)
- added MX3: NUMPAD_SLASH, picopad:MXOnly-1U-Hotswap, F.Cu at (132.9, 58.7)
- added MX4: NUMLOCK, picopad:MXOnly-1U-Hotswap, F.Cu at (113.9, 58.7)
- added MX5: NUMPAD_7, picopad:MXOnly-1U-Hotswap, F.Cu at (113.9, 77.7)
- added MX6: NUMPAD_8, picopad:MXOnly-1U-Hotswap, F.Cu at (132.9, 77.7)
- added MX7: NUMPAD_9, picopad:MXOnly-1U-Hotswap, F.Cu at (152.0, 77.7)
- added MX8: NUMPAD_PLUS, picopad:MXOnly-2U-Hotswap-Vertical, F.Cu at (171.0, 87.2)
- added MX9: NUMPAD_6, picopad:MXOnly-1U-Hotswap, F.Cu at (152.0, 96.8)
- added R1: 10k, Resistor_SMD:R_0805_2012Metric, B.Cu at (163.0, 69.5)
- added R2: 22, Resistor_SMD:R_0805_2012Metric, B.Cu at (124.4, 71.2)
- added R3: 22, Resistor_SMD:R_0805_2012Metric, B.Cu at (122.4, 71.2)
- added R4: 10k, Resistor_SMD:R_0805_2012Metric, B.Cu at (160.5, 92.8)
- added R5: 51k, Resistor_SMD:R_0805_2012Metric, B.Cu at (144.2, 49.3)
- added R6: 51k, Resistor_SMD:R_0805_2012Metric, B.Cu at (140.8, 49.3)
- added RGB1: WS2812B, picopad:WS2812B-3528, B.Cu at (171.0, 63.7)
- added RGB10: WS2812B, picopad:WS2812B-3528, B.Cu at (132.9, 101.8)
- added RGB11: WS2812B, picopad:WS2812B-3528, B.Cu at (113.9, 101.8)
- added RGB12: WS2812B, picopad:WS2812B-3528, B.Cu at (113.9, 120.8)
- added RGB13: WS2812B, picopad:WS2812B-3528, B.Cu at (132.9, 120.8)
- added RGB14: WS2812B, picopad:WS2812B-3528, B.Cu at (152.0, 120.8)
- added RGB15: WS2812B, picopad:WS2812B-3528, B.Cu at (171.0, 130.3)
- added RGB16: WS2812B, picopad:WS2812B-3528, B.Cu at (152.0, 139.9)
- added RGB17: WS2812B, picopad:WS2812B-3528, B.Cu at (123.4, 139.8)
- added RGB2: WS2812B, picopad:WS2812B-3528, B.Cu at (152.0, 63.7)
- added RGB3: WS2812B, picopad:WS2812B-3528, B.Cu at (132.9, 63.7)
- added RGB4: WS2812B, picopad:WS2812B-3528, B.Cu at (113.9, 63.7)
- added RGB5: WS2812B, picopad:WS2812B-3528, B.Cu at (113.9, 82.7)
- added RGB6: WS2812B, picopad:WS2812B-3528, B.Cu at (132.9, 82.7)
- added RGB7: WS2812B, picopad:WS2812B-3528, B.Cu at (152.0, 82.7)
- added RGB8: WS2812B, picopad:WS2812B-3528, B.Cu at (171.0, 92.2)
- added RGB9: WS2812B, picopad:WS2812B-3528, B.Cu at (152.0, 101.8)
- added SW1: SW_Push, Random-keyboard-parts:SKQG-1155865, B.Cu at (170.9, 71.7)
- added U1: ATmega32U4-AU, Package_QFP:TQFP-44_10x10mm_P0.8mm, B.Cu at (169.5, 106.3)
- added U2: PRTR5V0U2X, Random-keyboard-parts:SOT143B, B.Cu at (123.4, 67.2)
- added USB1: HRO-TYPE-C-31-M-12, Type-C:HRO-TYPE-C-31-M-12, B.Cu at (123.4, 42.7)
- added Y1: 16MHz, Crystal:Crystal_SMD_3225-4Pin_3.2x2.5mm, B.Cu at (171.0, 137.3)
Other:
- board outline added: 79 x 101.5 mm
